File: Electronics/Electronics.kicad_pcb (KiCad board)
At the start: 2 copper layers, 59 parts, among them J1 MOT_R, J3 MOT_L, P1 USB_C_Plug_USB2.0, SW1 RST, SW10 BTN8, SW11 BTN9, SW2 BOOT, SW3 BTN1, SW4 BTN2, SW5 BTN3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

Commit message: started routing
Parts:
- P1: footprint Connector_USB:USB_C_Receptacle_Molex_105450-0101 -> Connector_USB:USB_C_Receptacle_Palconn_UTC16-G
- moved BT1 288.7 mm to (190.1, 106.4), turned to -90 degrees
- moved J1 261.6 mm to (179.5, 81.1)
- moved J3 246.0 mm to (163.3, 81.2)
- moved U7 242.9 mm to (179.6, 102.7)
- moved U4 228.1 mm to (185.3, 92.8), turned to 90 degrees
- moved D1 227.7 mm to (126.6, 93.6), turned to 180 degrees
- moved R18 211.5 mm to (124.0, 93.6)
- moved BZ1 210.8 mm to (106.2, 113.6)
- moved U3 210.3 mm to (167.6, 93.5), turned to 90 degrees
- moved U6 197.9 mm to (133.3, 116.1), turned to -90 degrees
- moved U1 171.4 mm to (109.7, 95.6), turned to 90 degrees
- moved P1 166.8 mm to (123.3, 116.7)
- moved U5 27.2 mm to (-45.3, 131.2), turned to 180 degrees
Routing:
- net Net-(U6-VI): track 0.00 -> 6.15 mm
- net /STATUS: track 0.00 -> 1.57 mm
- net Net-(D1-A): track 0.00 -> 1.51 mm
Other:
- board outline added: 100 x 50 mm

Commit message: edging pcb done
Parts:
- J1, J3: footprint TerminalBlock_4Ucon:TerminalBlock_4Ucon_1x04_P3.50mm_Horizontal -> TerminalBlock_MetzConnect:TerminalBlock_MetzConnect_Type059_RT06304HBWC_1x04_P3.50mm_Horizontal
- moved SW8 288.1 mm to (188.2, 131.0)
- moved SW5 284.4 mm to (177.6, 135.1)
- moved SW4 284.1 mm to (177.4, 126.9)
- moved U8 277.3 mm to (172.7, 106.1)
- moved SW7 269.9 mm to (167.1, 130.8)
- moved SW3 261.4 mm to (152.5, 127.1)
- moved R9 251.0 mm to (158.8, 129.3)
- moved C15 247.1 mm to (194.0, 80.1), turned to 180 degrees
- moved C14 238.3 mm to (185.9, 89.9), turned to -90 degrees
- moved U2 238.2 mm to (133.7, 106.1)
- moved C4 232.7 mm to (176.1, 85.8), turned to -90 degrees
- moved C3 230.6 mm to (174.1, 87.6), turned to -90 degrees
- moved C5 227.5 mm to (170.5, 84.1), turned to 90 degrees
- moved SW1 225.2 mm to (122.2, 75.3)
- moved C18 225.0 mm to (176.2, 106.9), turned to 180 degrees
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Connections:
- BT1 pad 1: Net-(BT1-+) -> /BAT
- C14 pad 1: Net-(BT1-+) -> /BAT
- U7 pad 3: Net-(BT1-+) -> /BAT
Routing:
- net /SCL: track 0.00 -> 101.4 mm, vias 0 -> 4
- net /SDA: track 0.00 -> 85.8 mm, vias 0 -> 4
- net /STEP_R_STEP: track 0.00 -> 81.4 mm, vias 0 -> 2
- net /STEP_R_UART: track 0.00 -> 81.3 mm
- net /STEP_R_DIR: track 0.00 -> 81.0 mm, vias 0 -> 2
- net /SPREAD: track 0.00 -> 80.7 mm, vias 0 -> 4
- net /STEP_L_UART: track 0.00 -> 75.1 mm, vias 0 -> 2
- net /STEP_R_DIAG: track 0.00 -> 74.2 mm, vias 0 -> 2
- net /BTN5: track 0.00 -> 74.0 mm, vias 0 -> 2
- net /STEP_CURR: track 0.00 -> 72.6 mm, vias 0 -> 5
- net /STEP_L_DIR: track 0.00 -> 67.8 mm, vias 0 -> 2
- net /~{STEP_EN}: track 0.00 -> 65.8 mm, vias 0 -> 2
- net /STEP_L_STEP: track 0.00 -> 63.6 mm, vias 0 -> 2
- net /BTN1: track 0.00 -> 60.3 mm, vias 0 -> 2
- net /STEP_L_DIAG: track 0.00 -> 59.2 mm, vias 0 -> 2
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- added copper zone on F.Cu, net GND
Other:
- board size 100 x 50 mm -> 100 x 70 mm

Commit message: ready to manufacture, needs BOM, double checking
Parts:
- added G***: LOGO, LOGO, B.Cu at (180.4, 107.7)
- added G***: LOGO, LOGO, B.Cu at (112.4, 105.4)
- added G***: LOGO, LOGO, B.Cu at (148.7, 109.9)
- added G***: LOGO, LOGO, B.Cu at (189.4, 95.5)
- added G***: LOGO, LOGO, B.Cu at (145.7, 91.8)
- added G***: LOGO, LOGO, B.Cu at (170.3, 96.8)
- added G***: LOGO, LOGO, B.Cu at (192.3, 108.6)
- added G***: LOGO, LOGO, B.Cu at (138.0, 83.7)
- added G***: LOGO, LOGO, B.Cu at (120.7, 119.9)
- added G***: LOGO, LOGO, B.Cu at (131.5, 106.3)
- added G***: LOGO, LOGO, B.Cu at (138.8, 75.6)
- added G***: LOGO, LOGO, B.Cu at (178.7, 79.1)
- added G***: LOGO, LOGO, B.Cu at (114.3, 84.0)
- added G***: LOGO, LOGO, B.Cu at (178.7, 119.0)
- added G***: LOGO, LOGO, B.Cu at (155.0, 82.6)
- added G***: LOGO, LOGO, B.Cu at (115.6, 126.4)
- added G***: LOGO, LOGO, B.Cu at (131.7, 126.5)
- J1, J3: footprint TerminalBlock_MetzConnect:TerminalBlock_MetzConnect_Type059_RT06304HBWC_1x04_P3.50mm_Horizontal -> TerminalBlock_Phoenix:TerminalBlock_Phoenix_PT-1,5-4-3.5-H_1x04_P3.50mm_Horizontal
- SW1, SW10, SW11, SW2, SW3, SW4, SW5, SW6, SW7, SW8, SW9: footprint Button_Switch_SMD:SW_Push_1P1T_NO_6x6mm_H9.5mm -> Button_Switch_SMD:SW_Push_1P1T_NO_CK_KMR2
- moved R5 253.3 mm to (160.4, 118.1), turned to -90 degrees
- moved R3 253.2 mm to (160.6, 109.3), turned to 90 degrees
- moved R10 251.4 mm to (160.8, 115.2)
- moved R11 251.2 mm to (160.8, 114.0)
- moved R12 250.6 mm to (160.7, 107.8)
- moved R4 249.7 mm to (157.4, 102.2)
- moved R7 248.1 mm to (155.8, 100.7), turned to 90 degrees
- moved R13 244.3 mm to (154.5, 98.7), turned to 90 degrees
- moved R14 243.1 mm to (153.3, 101.9), turned to 90 degrees
- moved R2 233.2 mm to (139.8, 116.9), turned to 90 degrees
- moved C6 64.7 mm to (169.7, 119.0), turned to 180 degrees
- moved R15 64.4 mm to (152.0, 100.0), turned to 90 degrees
- moved SW1 61.7 mm to (164.9, 119.8), turned to 180 degrees
- moved R16 58.0 mm to (150.8, 101.8), turned to 90 degrees
- moved R6 53.1 mm to (160.4, 119.7), turned to -90 degrees
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Connections:
- U3 pad 29: (no net) -> GND
- U4 pad 29: (no net) -> GND
Routing:
- net VCC: track 13.2 -> 357.1 mm, vias 0 -> 17
- net GND: track 0.00 -> 105.8 mm, vias 0 -> 30
- net /BAT: track 49.3 -> 108.8 mm
- net /STEP_R_UART: track 81.3 -> 28.8 mm, vias 0 -> 2
- net /BTN4: track 7.95 -> 54.2 mm
- net /BTN7: track 9.70 -> 54.8 mm, vias 0 -> 2
- net /BTN5: track 74.0 -> 30.0 mm
- net /BTN9: track 9.76 -> 52.3 mm, vias 0 -> 2
- net /STEP_R_STEP: track 81.4 -> 39.0 mm
- net /STEP_L_UART: track 75.1 -> 33.7 mm
- net /BTN1: track 60.3 -> 20.0 mm, vias 2 -> 0
- net /STEP_R_DIAG: track 74.2 -> 35.1 mm, vias 2 -> 4
- net Net-(U1-EN): track 49.0 -> 10.4 mm, vias 2 -> 0
- net /STEP_R_DIR: track 81.0 -> 42.9 mm
- net /STEP_L_STEP: track 63.6 -> 25.8 mm
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- added copper zone on B.Cu, net GND
Other:
- board size 100 x 70 mm -> 100 x 60 mm
- board text added: "STUYOLY TECH 2025 | Beter R.T PCB"

Commit message: production ready fr
Parts:
- BT1: footprint Connector_AMASS:AMASS_XT30UPB-F_1x02_P5.0mm_Vertical -> TerminalBlock_Phoenix:TerminalBlock_Phoenix_PT-1,5-2-3.5-H_1x02_P3.50mm_Horizontal
- C1, C11, C16, C17, C18, C19, C2, C3, C4, C6: footprint Capacitor_SMD:C_0603_1608Metric -> Capacitor_SMD:C_0402_1005Metric
- P1: footprint Connector_USB:USB_C_Receptacle_Palconn_UTC16-G -> Connector_USB:USB_C_Receptacle_GCT_USB4110
- moved BT1 3.79 mm to (195.3, 118.6), turned to 90 degrees
- moved C19 2.52 mm to (169.7, 99.6), turned to -90 degrees
- moved C13 2.30 mm to (180.6, 119.3)
- moved C12 2.00 mm to (190.3, 122.4)
- moved U6 1.90 mm to (187.1, 117.0)
- moved C16 1.32 mm to (141.0, 100.3), turned to -90 degrees
- moved C17 1.10 mm to (163.7, 104.2), turned to 180 degrees
- moved P1 0.58 mm to (181.6, 126.3)
- moved C18 0.33 mm to (132.9, 102.3)
- moved C4 0.20 mm to (153.7, 85.3)
Routing:
- net VCC: track 357.1 -> 363.1 mm
- net /BAT: track 108.8 -> 113.5 mm
- net GND: track 105.8 -> 101.5 mm, vias 30 -> 29
- net /SDA: track 101.9 -> 100.7 mm
- net /SCL: track 123.9 -> 125.0 mm
- net /STEP_R_UART: track 28.8 -> 28.0 mm
- net /SPREAD: track 49.9 -> 50.5 mm
