File: Electronics/Electronics.kicad_sch (KiCad schematic)
At the start: 54 parts, among them J1 MOT_L, J2 MOT_R, P1 USB_C_Plug_USB2.0, SW1 RST, SW10 BTN8, SW11 BTN9, SW2 BOOT, SW3 BTN1, SW4 BTN2, SW5 BTN3, SW6 BTN4, SW7 BTN5, SW8 BTN6, SW9 BTN7, U1 ESP32-S3-WROOM-1, U2 BMI270, U5 BMI270, U6 NCP1117-3.3_SOT223, U7 NCP1117-3.3_SOT223

Commit message: oleds
Parts:
- removed C10, C7, C8, C9: 100n, symbol Device:C
- removed U2, U5: BMI270, Package_LGA:Bosch_LGA-14_3x2.5mm_P0.5mm, symbol Sensor_Motion:BMI160
- added C16, C17, C18, C19: 100n, symbol Device:C
- added U2, U8: ~, Package_LGA:Bosch_LGA-14_3x2.5mm_P0.5mm, symbol BMI270:BMI270
- added U5, U9: ~, Connector_PinHeader_2.54mm:PinHeader_1x04_P2.54mm_Vertical, symbol 0.96InchOLED:0.96_Inch_OLED
Connections:
- net GND: now also C16.1, C17.1, C18.1, C19.1, U2.6 (GNDI0), U2.7 (GND), U5.1 (GND), U8.1 (SDO), U8.6 (GNDI0), U8.7 (GND), U9.1 (GND)
- net SCL: now also U2.13 (SCx), U5.3 (SDA), U8.13 (SCx), U9.3 (SDA)
- net SDA: now also U2.14 (SDx), U5.4 (SCL), U8.14 (SDx), U9.4 (SCL)
- net VCC: now also C16.2, C17.2, C18.2, C19.2, U2.1 (SDO), U2.12 (CSB), U2.5 (VDDI0), U2.8 (VDD), U5.2 (VCC), U8.12 (CSB), U8.5 (VDDI0), U8.8 (VDD), U9.2 (VCC)
Other:
- note added: "Battery"
- note added: "Buttons/Interface"
- note added: "Displays"
- note added: "ESP32"
- note added: "IMUs"
- note added: "Motor Drivers"
- note added: "USB"
- moved on the sheet: C11, C5, C6, R1, R10, R11, R12, R13, R14, R15, R16, R17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

Commit message: Schematics Done, footprints assigned
Parts:
- removed J1: MOT_L, symbol Connector:Conn_01x04_Pin
- removed J2: MOT_R, symbol Connector:Conn_01x04_Pin
- added BZ1: AI-1223, Buzzer_Beeper:Buzzer_12x9.5RM7.6, symbol Device:Buzzer
- added D1: STATUS_LED, LED_SMD:LED_0603_1608Metric, symbol Device:LED
- added J1: MOT_R, TerminalBlock_4Ucon:TerminalBlock_4Ucon_1x04_P3.50mm_Horizontal, symbol Connector:Screw_Terminal_01x04
- added J3: MOT_L, TerminalBlock_4Ucon:TerminalBlock_4Ucon_1x04_P3.50mm_Horizontal, symbol Connector:Screw_Terminal_01x04
- added R18: 1k, Resistor_SMD:R_0201_0603Metric, symbol Device:R
- BT1: footprint (none) -> Connector_AMASS:AMASS_XT30UPB-F_1x02_P5.0mm_Vertical
- C1, C11, C12, C13, C14, C15, C16, C17, C18, C19, C2, C3, C4, C5, C6: footprint (none) -> Capacitor_SMD:C_0603_1608Metric
- P1: footprint (none) -> Connector_USB:USB_C_Receptacle_Molex_105450-0101
- R1, R10, R11, R12, R13, R14, R15, R16, R17, R2, R3, R4, R5, R6, R7, R8, R9: footprint (none) -> Resistor_SMD:R_0201_0603Metric
- SW1, SW10, SW11, SW2, SW3, SW4, SW5, SW6, SW7, SW8, SW9: footprint (none) -> Button_Switch_SMD:SW_Push_1P1T_NO_6x6mm_H9.5mm
Connections:
- net GND: now also BZ1.2 (-), D1.1 (K)
- net at U4.1 (OB2): now also J1.4 (Pin_4)
- net at U4.21 (OA2): now also J1.2 (Pin_2)
- net at U4.24 (OA1): now also J1.1 (Pin_1)
- net at U4.26 (OB1): now also J1.3 (Pin_3)
- net at U3.1 (OB2): now also J3.4 (Pin_4)
- net at U3.26 (OB1): now also J3.3 (Pin_3)
- net at U3.21 (OA2): now also J3.2 (Pin_2)
- net at U3.24 (OA1): now also J3.1 (Pin_1)
- net STATUS: now reaches U1.22 (IO14)
- net STATUS: now also R18.1
- net BUZZ: now reaches U1.35 (IO42)
- net BUZZ: now also BZ1.1 (+)
- new net: D1.2 (A), R18.2
- no-connect marks 28 -> 26
Other:
- note added: "Buzzer"
- note added: "Status LED"

Commit message: started routing
Parts:
- P1: footprint Connector_USB:USB_C_Receptacle_Molex_105450-0101 -> Connector_USB:USB_C_Receptacle_Palconn_UTC16-G
Changed lines of the file:
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@@
 			)
 		)
-		(property "Footprint" "Connector_USB:USB_C_Receptacle_Molex_105450-0101"
+		(property "Footprint" "Connector_USB:USB_C_Receptacle_Palconn_UTC16-G"
 			(at 30.48 38.1 0)
 			(effects

Commit message: edging pcb done
Parts:
- J1, J3: footprint TerminalBlock_4Ucon:TerminalBlock_4Ucon_1x04_P3.50mm_Horizontal -> TerminalBlock_MetzConnect:TerminalBlock_MetzConnect_Type059_RT06304HBWC_1x04_P3.50mm_Horizontal
Connections:
- net BAT: now also BT1.1 (+), C14.1, U7.3 (VI)
Changed lines of the file:
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@@
 	)
 	(junction
+		(at 87.63 22.86)
+		(diameter 0)
+		(color 0 0 0 0)
+	)
+	(junction
 		(at 261.62 123.19)
 		(diameter 0)
@@
 	(wire
 		(pts
-			(xy 87.63 22.86) (xy 104.14 22.86)
+			(xy 83.82 22.86) (xy 87.63 22.86)
 		)
 		(stroke
@@
 	(wire
 		(pts
+			(xy 87.63 22.86) (xy 87.63 25.4)
+		)
+		(stroke
+			(width 0)
+			(type default)
+		)
+	)
+	(wire
+		(pts
 			(xy 66.04 154.94) (xy 73.66 154.94)
 		)
@@
 	(wire
 		(pts
+			(xy 87.63 22.86) (xy 104.14 22.86)
+		)
+		(stroke
+			(width 0)
+			(type default)
+		)
+	)
+	(wire
+		(pts
 			(xy 33.02 100.33) (xy 33.02 102.87)
 		)
@@
 	(wire
 		(pts
-			(xy 87.63 22.86) (xy 87.63 25.4)
-		)
-		(stroke
-			(width 0)
-			(type default)
-		)
-	)
-	(wire
-		(pts
 			(xy 138.43 66.04) (xy 138.43 20.32)
 		)
@@
 		)
 	)
+	(label "BAT"
+		(at 83.82 22.86 0)
+		(effects
+			(font
+				(size 1.27 1.27)
+			)
+			(justify left bottom)
+		)
+	)
 	(label "BTN9"
 		(at 66.04 172.72 0)
@@
 			)
 		)
-		(property "Footprint" "TerminalBlock_4Ucon:TerminalBlock_4Ucon_1x04_P3.50mm_Horizontal"
+		(property "Footprint" "TerminalBlock_MetzConnect:TerminalBlock_MetzConnect_Type059_RT06304HBWC_1x04_P3.50mm_Horizontal"
 			(at 275.59 39.37 0)
 			(effects
@@
 			)
 		)
-		(property "Footprint" "TerminalBlock_4Ucon:TerminalBlock_4Ucon_1x04_P3.50mm_Horizontal"
+		(property "Footprint" "TerminalBlock_MetzConnect:TerminalBlock_MetzConnect_Type059_RT06304HBWC_1x04_P3.50mm_Horizontal"
 			(at 203.2 39.37 0)
 			(effects

Commit message: ready to manufacture, needs BOM, double checking
Parts:
- J1, J3: footprint TerminalBlock_MetzConnect:TerminalBlock_MetzConnect_Type059_RT06304HBWC_1x04_P3.50mm_Horizontal -> TerminalBlock_Phoenix:TerminalBlock_Phoenix_PT-1,5-4-3.5-H_1x04_P3.50mm_Horizontal
- SW1, SW10, SW11, SW2, SW3, SW4, SW5, SW6, SW7, SW8, SW9: footprint Button_Switch_SMD:SW_Push_1P1T_NO_6x6mm_H9.5mm -> Button_Switch_SMD:SW_Push_1P1T_NO_CK_KMR2
Connections:
- net GND: now also U3.29 (GND), U4.29 (GND)

Commit message: production ready fr
Parts:
- BT1: footprint Connector_AMASS:AMASS_XT30UPB-F_1x02_P5.0mm_Vertical -> TerminalBlock_Phoenix:TerminalBlock_Phoenix_PT-1,5-2-3.5-H_1x02_P3.50mm_Horizontal
- C1, C11, C16, C17, C18, C19, C2, C3, C4, C6: footprint Capacitor_SMD:C_0603_1608Metric -> Capacitor_SMD:C_0402_1005Metric
- P1: footprint Connector_USB:USB_C_Receptacle_Palconn_UTC16-G -> Connector_USB:USB_C_Receptacle_GCT_USB4110
Changed lines of the file:
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@@
 			)
 		)
-		(property "Footprint" "Capacitor_SMD:C_0603_1608Metric"
+		(property "Footprint" "Capacitor_SMD:C_0402_1005Metric"
 			(at 267.0048 135.89 0)
 			(effects
@@
 			)
 		)
-		(property "Footprint" "Capacitor_SMD:C_0603_1608Metric"
+		(property "Footprint" "Capacitor_SMD:C_0402_1005Metric"
 			(at 224.4852 34.29 0)
 			(effects
@@
 			)
 		)
-		(property "Footprint" "Capacitor_SMD:C_0603_1608Metric"
+		(property "Footprint" "Capacitor_SMD:C_0402_1005Metric"
 			(at 152.0952 34.29 0)
 			(effects
@@
 			)
 		)
-		(property "Footprint" "Capacitor_SMD:C_0603_1608Metric"
+		(property "Footprint" "Capacitor_SMD:C_0402_1005Metric"
 			(at 260.6548 135.89 0)
 			(effects
@@
 			)
 		)
-		(property "Footprint" "Capacitor_SMD:C_0603_1608Metric"
+		(property "Footprint" "Capacitor_SMD:C_0402_1005Metric"
 			(at 51.1048 152.4 0)
 			(effects
@@
 			)
 		)
-		(property "Footprint" "Capacitor_SMD:C_0603_1608Metric"
+		(property "Footprint" "Capacitor_SMD:C_0402_1005Metric"
 			(at 279.7048 135.89 0)
 			(effects
@@
 			)
 		)
-		(property "Footprint" "Capacitor_SMD:C_0603_1608Metric"
+		(property "Footprint" "Capacitor_SMD:C_0402_1005Metric"
 			(at 37.1348 137.16 0)
 			(effects
@@
 			)
 		)
-		(property "Footprint" "Capacitor_SMD:C_0603_1608Metric"
+		(property "Footprint" "Capacitor_SMD:C_0402_1005Metric"
 			(at 199.39 63.5 0)
 			(effects
@@
 			)
 		)
-		(property "Footprint" "Connector_AMASS:AMASS_XT30UPB-F_1x02_P5.0mm_Vertical"
+		(property "Footprint" "TerminalBlock_Phoenix:TerminalBlock_Phoenix_PT-1,5-2-3.5-H_1x02_P3.50mm_Horizontal"
 			(at 87.63 28.956 90)
 			(effects
@@
 			)
 		)
-		(property "Footprint" "Connector_USB:USB_C_Receptacle_Palconn_UTC16-G"
+		(property "Footprint" "Connector_USB:USB_C_Receptacle_GCT_USB4110"
 			(at 30.48 38.1 0)
 			(effects
@@
 			)
 		)
-		(property "Footprint" "Capacitor_SMD:C_0603_1608Metric"
+		(property "Footprint" "Capacitor_SMD:C_0402_1005Metric"
 			(at 273.3548 135.89 0)
 			(effects
@@
 			)
 		)
-		(property "Footprint" "Capacitor_SMD:C_0603_1608Metric"
+		(property "Footprint" "Capacitor_SMD:C_0402_1005Metric"
 			(at 271.78 63.5 0)
 			(effects
