File: Electronics V2/Electronics V2.kicad_pcb (KiCad board)
At the start: 2 copper layers, 102 x 62 mm, 86 parts, among them J1 MOT_L, J2 MOT_R, J3 SD_Card, J4 USB_C_Receptacle_USB2.0_14P, J5 Power Probes, SW1 BTN_0, SW2 MSTP_SEL, SW3 RST, SW4 BOOT, SW5 BTN_1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

Commit message: routed power, etc
Parts:
- added J6: L1, TerminalBlock_Phoenix:TerminalBlock_Phoenix_PT-1,5-2-3.5-H_1x02_P3.50mm_Horizontal, F.Cu at (135.4, 71.2)
- added J7: L2, TerminalBlock_Phoenix:TerminalBlock_Phoenix_PT-1,5-2-3.5-H_1x02_P3.50mm_Horizontal, F.Cu at (143.9, 71.2)
- added Q1: BC547, Package_TO_SOT_THT:TO-92_Inline, F.Cu at (140.1, 80.3)
- J3: moved to B.Cu
- moved C4 164.4 mm to (186.1, 82.2), turned to -90 degrees
- moved SW8 139.2 mm to (190.2, 115.2), turned to 90 degrees
- moved D2 137.0 mm to (182.4, 123.7)
- moved BT1 132.6 mm to (190.5, 123.4)
- moved U2 129.1 mm to (158.2, 83.5)
- moved SW2 127.9 mm to (150.5, 81.9), turned to 90 degrees
- moved U9 127.2 mm to (179.4, 83.5)
- moved SW9 126.3 mm to (172.0, 81.9), turned to 90 degrees
- moved C9 121.4 mm to (164.5, 82.2), turned to -90 degrees
- moved J5 118.9 mm to (199.4, 79.3)
- moved U7 118.7 mm to (186.5, 93.5)
- moved U10 118.0 mm to (183.3, 115.5), turned to 180 degrees
- moved R24 115.9 mm to (195.3, 79.3)
- moved R22 106.6 mm to (153.8, 120.8)
- moved SW6 103.9 mm to (176.3, 112.9), turned to 90 degrees
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Connections:
- BT1 pad 1: VBAT -> Net-(BT1-+)
- C21 pad 1: Net-(D2-K) -> VBAT
- D2 pad 1: Net-(D2-K) -> VBAT
- D2 pad 2: VBAT -> Net-(BT1-+)
- U10 pad 4: Net-(D2-K) -> VBAT
- U10 pad 5: Net-(D2-K) -> VBAT
- U10 pad 6: Net-(D2-K) -> VBAT
- U7 pad 3: Net-(D2-K) -> VBAT
Routing:
- net VBAT: track 0.00 -> 112.0 mm
- net /D-: track 0.00 -> 18.7 mm
- net /D+: track 0.00 -> 18.5 mm
- net Net-(BT1-+): track 0.00 -> 8.10 mm
- net /SD_DETECT: track 0.00 -> 3.30 mm, vias 0 -> 1
Other:
- outline, holes or cut-outs redrawn

Commit message: placing done
Parts:
- removed SW9: MSTP_SEL, Button_Switch_SMD:SW_DIP_SPSTx02_Slide_6.7x6.64mm_W6.73mm_P2.54mm_LowProfile_JPin
- moved C6 158.5 mm to (171.7, 69.9), turned to 90 degrees
- moved C5 156.2 mm to (170.1, 69.9), turned to 90 degrees
- moved R14 146.2 mm to (176.0, 126.1), turned to 90 degrees
- moved C15 139.3 mm to (177.8, 126.0), turned to 90 degrees
- moved C1 137.5 mm to (197.7, 82.3)
- moved C17 135.9 mm to (180.2, 122.7), turned to -90 degrees
- moved C13 133.3 mm to (197.7, 80.8)
- moved R3 133.0 mm to (146.2, 83.8)
- moved R2 132.7 mm to (145.8, 81.0), turned to 180 degrees
- moved R20 131.0 mm to (162.4, 76.1)
- moved C7 126.2 mm to (141.9, 85.5), turned to 180 degrees
- moved R4 126.0 mm to (135.1, 76.5), turned to 180 degrees
- moved C27 125.8 mm to (194.1, 84.9)
- moved R5 125.4 mm to (136.8, 84.8)
- moved R16 125.1 mm to (178.5, 122.7), turned to -90 degrees
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Connections:
- R2 pad 1: Net-(U2-MS1_AD1) -> /Motor Driver_L/MS1_AD1
- R3 pad 1: Net-(U2-MS1_AD0) -> /Motor Driver_L/MS1_AD0
- R6 pad 1: Net-(U9-MS1_AD1) -> /Motor Driver_L/MS1_AD0
- R7 pad 1: Net-(U9-MS1_AD0) -> /Motor Driver_L/MS1_AD1
- SW2 pad 3: Net-(U2-MS1_AD1) -> /Motor Driver_L/MS1_AD0
- SW2 pad 4: Net-(U2-MS1_AD0) -> /Motor Driver_L/MS1_AD1
- U2 pad 10: Net-(U2-MS1_AD1) -> /Motor Driver_L/MS1_AD1
- U2 pad 9: Net-(U2-MS1_AD0) -> /Motor Driver_L/MS1_AD0
- U3 pad 23: unconnected-(U3-IO21-Pad23) -> /LASER
- U3 pad 28: unconnected-(U3-IO35-Pad28) -> /MS1_AD1
- U3 pad 29: unconnected-(U3-IO36-Pad29) -> /MS1_AD0
- U9 pad 10: Net-(U9-MS1_AD1) -> /Motor Driver_L/MS1_AD0
- U9 pad 9: Net-(U9-MS1_AD0) -> /Motor Driver_L/MS1_AD1
Routing:
- net VBAT: track 112.0 -> 44.2 mm, vias 0 -> 8
- net /D-: track 18.7 -> 0.00 mm
- net /D+: track 18.5 -> 0.00 mm
- net +3V3: track 0.00 -> 11.8 mm
- net +5V: track 0.00 -> 11.4 mm
- net Net-(U7-VO): track 0.00 -> 11.3 mm
- net Net-(U3-EN): track 0.00 -> 8.64 mm
- net /SD_DETECT: track 3.30 -> 0.00 mm, vias 1 -> 0
- net /INCR_BTN: track 0.00 -> 0.50 mm
Other:
- outline, holes or cut-outs redrawn

Commit message: completed pcb (maybe)
Parts:
- moved R21 2.74 mm to (159.2, 113.9)
- moved D3 1.90 mm to (159.3, 115.6)
- moved C25 0.10 mm to (156.1, 76.1)
- moved C19 0.10 mm to (199.9, 100.9)
- moved R2 0.10 mm to (145.9, 81.0)
Connections:
- U3 pad 28: /MS1_AD1 -> unconnected-(U3-IO35-Pad28)
- U3 pad 29: /MS1_AD0 -> unconnected-(U3-IO36-Pad29)
Routing:
- net +3V3: track 11.8 -> 481.6 mm, vias 0 -> 30
- net +5V: track 11.4 -> 211.1 mm, vias 0 -> 6
- net /SCL: track 0.00 -> 163.6 mm, vias 0 -> 8
- net /SDA: track 0.00 -> 155.4 mm, vias 0 -> 6
- net VBAT: track 44.2 -> 156.4 mm, vias 8 -> 15
- net /INCR_B: track 0.00 -> 78.7 mm, vias 0 -> 6
- net /~{EN}: track 0.00 -> 68.5 mm, vias 0 -> 3
- net /INCR_A: track 0.00 -> 68.5 mm, vias 0 -> 4
- net /BTN_0: track 0.00 -> 66.2 mm, vias 0 -> 2
- net /INCR_BTN: track 0.50 -> 61.2 mm, vias 0 -> 2
- net /BTN_2: track 0.00 -> 57.4 mm
- net /VREF: track 0.00 -> 53.3 mm, vias 0 -> 5
- net GND: track 0.00 -> 51.3 mm, vias 0 -> 16
- net /DIAG_L: track 0.00 -> 47.9 mm, vias 0 -> 4
- net /SPREAD: track 0.00 -> 46.5 mm, vias 0 -> 3
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- added copper zone on B.Cu, net GND
- added copper zone on F.Cu, net GND
