File: Electronics V2/Electronics V2.kicad_pcb (KiCad board)
At the start: 2 copper layers, 102 x 62 mm, 88 parts, among them J1 MOT_L, J2 MOT_R, J3 SD_Card, J4 USB_C_Receptacle_USB2.0_14P, J5 Power Probes, J6 L1, J7 L2, Q1 BC547, SW1 BTN_0, SW2 MSTP_SEL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

Commit message: finish routing jit
Parts:
- removed R6, R7: 10k, Resistor_SMD:R_0603_1608Metric
- moved D2 147.6 mm to (196.6, 91.8), turned to 90 degrees
- moved J5 144.7 mm to (197.9, 104.5), turned to 180 degrees
- moved C21 143.9 mm to (188.9, 93.6), turned to -90 degrees
- moved D1 142.6 mm to (180.0, 123.5), turned to 180 degrees
- moved C19 141.1 mm to (188.5, 111.0), turned to 90 degrees
- moved D3 140.2 mm to (180.0, 121.7), turned to 180 degrees
- moved D5 139.0 mm to (191.3, 102.0)
- moved D6 138.9 mm to (191.3, 104.5)
- moved C20 136.6 mm to (183.3, 103.3), turned to 180 degrees
- moved SW3 135.7 mm to (181.4, 126.3)
- moved R24 135.3 mm to (194.4, 104.5)
- moved R23 135.3 mm to (194.4, 102.0)
- moved C13 134.7 mm to (177.3, 102.2), turned to -90 degrees
- moved C12 133.0 mm to (176.0, 126.2), turned to 90 degrees
- moved U11 129.0 mm to (190.7, 110.8), turned to -90 degrees
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Connections:
- C12 pad 1: +3V3 -> Net-(U3-EN)
- C22 pad 1: Net-(U7-VO) -> +3V3
- J1 pad 1: /Motor Driver_L/A1 -> /Motor Driver_L/A2
- J1 pad 2: /Motor Driver_L/A2 -> /Motor Driver_L/A1
- J2 pad 1: /Motor Driver_R/A1 -> /Motor Driver_R/A2
- J2 pad 2: /Motor Driver_R/A2 -> /Motor Driver_R/A1
- Q1 pad 1: +3V3 -> +5V
- SW2 pad 3: /Motor Driver_L/MS1_AD0 -> /Motor Driver_L/MS1_AD1
- SW2 pad 4: /Motor Driver_L/MS1_AD1 -> /Motor Driver_L/MS1_AD0
- U7 pad 2: Net-(U7-VO) -> +3V3
- U9 pad 10: /Motor Driver_L/MS1_AD0 -> /Motor Driver_L/MS1_AD1
- U9 pad 9: /Motor Driver_L/MS1_AD1 -> /Motor Driver_L/MS1_AD0
Routing:
- net +3V3: track 0.00 -> 76.2 mm
- net VBAT: track 0.00 -> 69.5 mm, vias 0 -> 4
- net /Motor Driver_L/MS1_AD1: track 0.00 -> 32.4 mm, vias 0 -> 2
- net /Motor Driver_L/MS1_AD0: track 0.00 -> 31.2 mm, vias 0 -> 2
- net /VREF: track 0.00 -> 28.8 mm
- net +5V: track 0.00 -> 25.8 mm
- net /D+: track 0.00 -> 22.8 mm
- net /D-: track 0.00 -> 22.8 mm
- net Net-(J6-Pin_1): track 0.00 -> 19.7 mm
- net /Motor Driver_R/A2: track 0.00 -> 17.6 mm, vias 0 -> 1
- net /Motor Driver_L/A2: track 0.00 -> 17.0 mm, vias 0 -> 1
- net /Motor Driver_L/A1: track 0.00 -> 14.3 mm
- net /Motor Driver_R/A1: track 0.00 -> 13.5 mm
- net /Motor Driver_R/B2: track 0.00 -> 13.1 mm, vias 0 -> 1
- net /Motor Driver_L/B2: track 0.00 -> 13.1 mm, vias 0 -> 1
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