File: Electronics V2/Electronics V2.kicad_sch (KiCad schematic)
At the start: 67 parts, among them J1 MOT_L, J2 MOT_R, J3 SD_Card, J4 USB_C_Receptacle_USB2.0_14P, J5 Power Probes, J6 L1, J7 L2, Q1 BC547, SW1 BTN_0, SW3 RST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

Commit message: routed power, etc
Connections:
- net VBAT: now also C21.1, D2.1 (K), U10.4 (IN), U10.5 (IN), U10.6 (IN), U7.3 (VI); no longer BT1.1 (+), D2.2 (A)
- new net: BT1.1 (+), D2.2 (A)
Changed lines of the file:
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@@
 	)
 	(junction
-		(at 17.78 81.28)
-		(diameter 0)
-		(color 0 0 0 0)
-	)
-	(junction
 		(at 105.41 157.48)
 		(diameter 0)
@@
 	(wire
 		(pts
+			(xy 43.18 78.74) (xy 43.18 81.28)
+		)
+		(stroke
+			(width 0)
+			(type default)
+		)
+	)
+	(wire
+		(pts
 			(xy 276.86 99.06) (xy 279.4 99.06)
 		)
@@
 	(wire
 		(pts
-			(xy 17.78 80.01) (xy 17.78 81.28)
-		)
-		(stroke
-			(width 0)
-			(type default)
-		)
-	)
-	(wire
-		(pts
 			(xy 111.76 133.35) (xy 111.76 128.27)
 		)
@@
 	)
 	(symbol
-		(lib_id "power:VCC")
-		(at 17.78 80.01 0)
-		(unit 1)
-		(exclude_from_sim no)
-		(in_bom yes)
-		(on_board yes)
-		(dnp no)
-		(property "Reference" "#PWR027"
-			(at 17.78 83.82 0)
-			(effects
-				(font
-					(size 1.27 1.27)
-				)
-				(hide yes)
-			)
-		)
-		(property "Value" "VBAT"
-			(at 17.78 76.454 0)
-			(effects
-				(font
-					(size 1.27 1.27)
-				)
-			)
-		)
-		(property "Footprint" ""
-			(at 17.78 80.01 0)
-			(effects
-				(font
-					(size 1.27 1.27)
-				)
-				(hide yes)
-			)
-		)
-		(property "Datasheet" ""
-			(at 17.78 80.01 0)
-			(effects
-				(font
-					(size 1.27 1.27)
-				)
-				(hide yes)
-			)
-		)
-		(property "Description" "Power symbol creates a global label with name \"VCC\""
-			(at 17.78 80.01 0)
-			(effects
-				(font
-					(size 1.27 1.27)
-				)
-				(hide yes)
-			)
-		)
-		(pin "1"
-		)
-		(instances
-			(project ""
-				(path "/fb299ee1-36f2-498d-9da8-1c8d846ea71b"
-					(reference "#PWR027")
-					(unit 1)
-				)
-			)
-		)
-	)
-	(symbol
 		(lib_id "Device:C")
 		(at 140.97 146.05 0)
@@
 					(unit 1)
 				)
+			)
+		)
+	)
+	(symbol
+		(lib_id "power:VCC")
+		(at 43.18 78.74 0)
+		(unit 1)
+		(exclude_from_sim no)
+		(in_bom yes)
+		(on_board yes)
+		(dnp no)
+		(property "Reference" "#PWR036"
+			(at 43.18 82.55 0)
+			(effects
+				(font
+					(size 1.27 1.27)
+				)
+				(hide yes)
+			)
+		)
+		(property "Value" "VBAT"
+			(at 43.18 75.184 0)
+			(effects
+				(font
+					(size 1.27 1.27)
+				)
+			)
+		)
+		(property "Footprint" ""
+			(at 43.18 78.74 0)
+			(effects
+				(font
+					(size 1.27 1.27)
+				)
+				(hide yes)
+			)
+		)
+		(property "Datasheet" ""
+			(at 43.18 78.74 0)
+			(effects
+				(font
+					(size 1.27 1.27)
+				)
+				(hide yes)
+			)
+		)
+		(property "Description" "Power symbol creates a global label with name \"VCC\""
+			(at 43.18 78.74 0)
+			(effects
+				(font
+					(size 1.27 1.27)
+				)
+				(hide yes)
+			)
+		)
+		(pin "1"
+		)
+		(instances
+			(project "Electronics V2"
+				(path "/fb299ee1-36f2-498d-9da8-1c8d846ea71b"
+					(reference "#PWR036")
+					(unit 1)
+				)

Commit message: placing done
Parts:
- added SW2: MSTP_SEL, Button_Switch_SMD:SW_DIP_SPSTx02_Slide_6.7x6.64mm_W6.73mm_P2.54mm_LowProfile_JPin, symbol Switch:SW_DIP_x02
Connections:
- net +3V3: now also SW2.1, SW2.2
- net LASER: now also U3.23 (IO21)
- net MS1_AD1: now reaches U3.28 (IO35)
- net MS1_AD0: now reaches U3.29 (IO36)
- new net Motor Driver_L/MS1_AD0: SW2.3
- new net Motor Driver_L/MS1_AD1: SW2.4
- no-connect marks 23 -> 20
Other:
- sheet Motor Driver_L ports: added MS1_AD0, MS1_AD1; removed none
- sheet Motor Driver_R ports: added MS1_AD0, MS1_AD1; removed none
- moved on the sheet: J1, J2

Commit message: completed pcb (maybe)
Connections:
- net MS1_AD0: no longer names the net of U3.29 (IO36)
- net MS1_AD1: no longer names the net of U3.28 (IO35)
- no-connect marks 20 -> 22
Changed lines of the file:
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@@
 	)
 	(no_connect
+		(at 181.61 50.8)
+	)
+	(no_connect
 		(at 52.07 166.37)
 	)
@@
 	)
 	(no_connect
+		(at 181.61 48.26)
+	)
+	(no_connect
 		(at 26.67 168.91)
 	)
@@
 	(wire
 		(pts
-			(xy 181.61 48.26) (xy 201.93 48.26)
-		)
-		(stroke
-			(width 0)
-			(type default)
-		)
-	)
-	(wire
-		(pts
 			(xy 218.44 36.83) (xy 228.6 36.83)
 		)
@@
 	(wire
 		(pts
-			(xy 181.61 50.8) (xy 201.93 50.8)
-		)
-		(stroke
-			(width 0)
-			(type default)
-		)
-	)
-	(wire
-		(pts
 			(xy 115.57 50.8) (xy 115.57 82.55)
 		)
@@
 		)
 	)
-	(label "MS1_AD1"
-		(at 201.93 48.26 180)
-		(effects
-			(font
-				(size 1.27 1.27)
-			)
-			(justify right bottom)
-		)
-	)
 	(label "MOSI"
 		(at 91.44 129.54 180)
@@
 		)
 	)
-	(label "MS1_AD0"
-		(at 201.93 50.8 180)
-		(effects
-			(font
-				(size 1.27 1.27)
-			)
-			(justify right bottom)
-		)
-	)

Commit message: finish routing jit
Parts:
- added R2, R3: 10k, Resistor_SMD:R_0603_1608Metric, symbol Device:R
Connections:
- net +3V3: now also C22.1, U7.2 (VO); no longer C12.1, Q1.1 (C)
- net +5V: now also Q1.1 (C)
- net GND: now also R2.1, R3.1
- net Motor Driver_L/A1: now also J1.2 (Pin_2); no longer J1.1 (Pin_1)
- net Motor Driver_L/A2: now also J1.1 (Pin_1); no longer J1.2 (Pin_2)
- net Motor Driver_L/MS1_AD0: now also SW2.4, R3.2; no longer SW2.3
- net Motor Driver_L/MS1_AD1: now also SW2.3, R2.2; no longer SW2.4
- net Motor Driver_R/A1: now also J2.2 (Pin_2); no longer J2.1 (Pin_1)
- net Motor Driver_R/A2: now also J2.1 (Pin_1); no longer J2.2 (Pin_2)
- net at R9.2, SW3.2, U3.3 (EN): now also C12.1

Commit message: needs review
Connections:
- net DIAG_L: now also U3.25 (IO48); no longer U3.35 (IO42)
- net DIAG_R: now also U3.21 (IO13); no longer U3.25 (IO48)
- net DIR_L: now also U3.22 (IO14); no longer U3.19 (IO11)
- net DIR_R: now also U3.18 (IO10); no longer U3.21 (IO13)
- net INDEX_R: now also U3.20 (IO12); no longer U3.26 (IO45)
- net LASER: now also U3.35 (IO42); no longer U3.23 (IO21)
- net SPREAD: now also U3.26 (IO45); no longer U3.22 (IO14)
- net STEP_L: now also U3.23 (IO21); no longer U3.18 (IO10)
- net STEP_R: now also U3.19 (IO11); no longer U3.20 (IO12)
Changed lines of the file:
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@@
 		)
 	)
-	(label "DIR_L"
+	(label "STEP_R"
 		(at 140.97 63.5 0)
 		(effects
@@
 		)
 	)
-	(label "DIAG_R"
+	(label "DIAG_L"
 		(at 204.47 76.2 180)
 		(effects
@@
 		)
 	)
-	(label "STEP_R"
+	(label "INDEX_R"
 		(at 140.97 66.04 0)
 		(effects
@@
 		)
 	)
-	(label "STEP_L"
+	(label "DIR_R"
 		(at 140.97 60.96 0)
 		(effects
@@
 		)
 	)
+	(label "STEP_L"
+		(at 201.93 45.72 180)
+		(effects
+			(font
+				(size 1.27 1.27)
+			)
+			(justify right bottom)
+		)
+	)
 	(label "LASER"
-		(at 201.93 45.72 180)
-		(effects
-			(font
-				(size 1.27 1.27)
-			)
-			(justify right bottom)
-		)
-	)
-	(label "DIAG_L"
 		(at 204.47 66.04 180)
 		(effects
@@
 		)
 	)
-	(label "DIR_R"
+	(label "DIAG_R"
 		(at 140.97 68.58 0)
 		(effects
@@
 		)
 	)
-	(label "SPREAD"
+	(label "DIR_L"
 		(at 140.97 71.12 0)
 		(effects
@@
 		)
 	)
-	(label "INDEX_R"
+	(label "SPREAD"
 		(at 204.47 68.58 180)
 		(effects
